File: production/pcbs/right/right.kicad_pcb (KiCad board)
At the start: 2 copper layers, 90 x 71 mm, 43 parts, among them T1 Flactyl 4.2 (right)

Commit message: Update pcb to 4.2
Parts:
- T1: moved to F.Cu
Routing:
- net C4_R0: track 187.0 -> 0.00 mm, vias 6 -> 0
- net R0: track 3.77 -> 187.0 mm, vias 0 -> 6
- net C4_R1D: track 123.9 -> 9.80 mm, vias 6 -> 0
- net C1: track 3.77 -> 117.1 mm, vias 0 -> 3
- net P9: track 103.5 -> 0.00 mm
- net P8: track 101.5 -> 0.00 mm, vias 2 -> 0
- net RAW: track 3.77 -> 103.5 mm
- net C4: track 143.6 -> 45.8 mm
- net R3: track 3.77 -> 101.5 mm, vias 0 -> 2
- net P0: track 75.4 -> 0.00 mm, vias 2 -> 0
- net P1: track 74.4 -> 0.00 mm, vias 4 -> 0
- net three: track 74.4 -> 0.00 mm, vias 1 -> 0
- net P3: track 3.77 -> 75.4 mm, vias 0 -> 2
- net P2: track 3.77 -> 74.4 mm, vias 0 -> 4
- net C3: track 9.80 -> 74.4 mm, vias 0 -> 1
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Other:
- net class Default removed
