File: production/pcbs/thumb/thumb.kicad_pcb (KiCad board)
At the start: 2 copper layers, 36 x 51 mm, 18 parts, among them T1 Flactyl 4.2 (thumb), T2 x, T3 y

Commit message: Update pcb to 4.2
Parts:
- T1, T2, T3: moved to F.Cu
Routing:
- net x: track 62.7 -> 0.00 mm
- net y: track 54.8 -> 0.00 mm
- net C6: track 3.77 -> 54.8 mm
- net R2: track 29.7 -> 62.7 mm
- net R1: track 3.77 -> 29.7 mm
- net Flactyl 4.2 (thumb): track 3.77 -> 0.00 mm
- net C6_R0D: track 0.00 -> 3.77 mm
- net C5_R2D: track 0.00 -> 3.77 mm
- net C6_R2D: track 0.00 -> 3.77 mm
- net C6_R1D: track 0.00 -> 3.77 mm
- net C5_R0: track 3.77 -> 0.00 mm
Other:
- net class Default removed
