File: production/pcbs/5.0/left/left.kicad_pcb (KiCad board)
At the start: 2 copper layers, 90 x 71 mm, 43 parts, among them T1 Flactyl 5.0 (left)

Commit message: V5 pcbs
Parts:
- moved SS1 0.25 mm to (20.5, -27.2)
Routing:
- net C4_R1D: track 131.2 -> 120.5 mm
- added copper zone on B.Cu, net GND
- added copper zone on F.Cu, net GND
Changed lines of the file:
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@@
     (footprint "SW-SMD_SS-3235D-03-L2.00" (layer "B.Cu")
     (attr smd)
-    (at 20.5 -27.5 0)
+    (at 20.5 -27.25 0)
     (fp_text reference "SS1" (at -0.087 -4.366) hide (layer "B.SilkS")
         (effects (font (size 1.143 1.143) (thickness 0.152)) (justify left))
@@
   (via (at 34.3 -40.1) (size 0.8) (drill 0.4) (layers "F.Cu" "B.Cu") (net 5))
   (via (at 74.8 -26.6) (size 0.8) (drill 0.4) (layers "F.Cu" "B.Cu") (net 5))
-  (segment (start 30 -30.5) (end 25.15 -30.5) (width 0.25) (layer "B.Cu") (net 5))
   (segment (start 33.4 -29.7) (end 32.8 -30.3) (width 0.25) (layer "B.Cu") (net 5))
   (segment (start 32.75 -30.25) (end 32.8 -30.3) (width 0.25) (layer "B.Cu") (net 5))
@@
   (segment (start 74.99 -30.69) (end 74.9 -30.6) (width 0.25) (layer "B.Cu") (net 5))
   (segment (start 2.6 -35.4) (end 13.9 -35.4) (width 0.25) (layer "B.Cu") (net 5))
+  (segment (start 18.8 -36.6) (end 23.361241 -32.038759) (width 0.25) (layer "B.Cu") (net 5))
+  (segment (start 15.1 -36.6) (end 18.8 -36.6) (width 0.25) (layer "B.Cu") (net 5))
   (segment (start 56.9 -28.4) (end 57.575 -29.075) (width 0.25) (layer "B.Cu") (net 5))
-  (segment (start 25.15 -30.5) (end 23.15 -28.5) (width 0.25) (layer "B.Cu") (net 5))
+  (segment (start 23.361241 -31.593758) (end 24.306242 -31.593758) (width 0.25) (layer "B.Cu") (net 5))
   (segment (start 2.475 -35.275) (end 2.6 -35.4) (width 0.25) (layer "B.Cu") (net 5))
   (segment (start 13.9 -35.4) (end 15.1 -36.6) (width 0.25) (layer "B.Cu") (net 5))
-  (segment (start 23.15 -28.5) (end 2.475 -28.5) (width 0.25) (layer "B.Cu") (net 5))
+  (segment (start 24.306242 -31.593758) (end 25.4 -30.5) (width 0.25) (layer "B.Cu") (net 5))
   (segment (start -2.9 -19.6) (end -0.69835 -19.6) (width 0.25) (layer "B.Cu") (net 5))
   (segment (start 74.8 -26.6) (end 74.8 -25.5) (width 0.25) (layer "B.Cu") (net 5))
+  (segment (start 23.361241 -32.038759) (end 23.361241 -31.593758) (width 0.25) (layer "B.Cu") (net 5))
   (segment (start 56.9 -28.4) (end 52 -28.4) (width 0.25) (layer "B.Cu") (net 5))
   (segment (start 30 -30.5) (end 32.5 -30.5) (width 0.25) (layer "B.Cu") (net 5))
@@
   (segment (start 74.8 -25.5) (end 74.9 -25.4) (width 0.25) (layer "B.Cu") (net 5))
   (segment (start 79.62 -30.69) (end 74.99 -30.69) (width 0.25) (layer "B.Cu") (net 5))
+  (segment (start 25.4 -30.5) (end 30 -30.5) (width 0.25) (layer "B.Cu") (net 5))
   (segment (start 34.3 -40.1) (end 33.6 -40.1) (width 0.25) (layer "B.Cu") (net 5))
   (segment (start 63.6887 -26.8113) (end 66.0887 -26.8113) (width 0.25) (layer "B.Cu") (net 5))
@@
   (via (at 24.4 -52.9504) (size 0.8) (drill 0.4) (layers "F.Cu" "B.Cu") (net 15))
   (via (at 61.9 -52.5) (size 0.8) (drill 0.4) (layers "F.Cu" "B.Cu") (net 15))
-  (segment (start 14.475 -29.275) (end 18.794294 -29.275) (width 0.25) (layer "B.Cu") (net 15))
+  (segment (start 21.413357 -31.613357) (end 21.413357 -31.894063) (width 0.25) (layer "B.Cu") (net 15))
   (segment (start 61.875 -52.525) (end 61.9 -52.5) (width 0.25) (layer "B.Cu") (net 15))
   (segment (start 34.369101 -52.6759) (end 35.134501 -51.9105) (width 0.25) (layer "B.Cu") (net 15))
   (segment (start 38.725 -52.525) (end 61.875 -52.525) (width 0.25) (layer "B.Cu") (net 15))
+  (segment (start 14.725 -29.025) (end 18.825 -29.025) (width 0.25) (layer "B.Cu") (net 15))
   (segment (start 24.6745 -52.6759) (end 34.369101 -52.6759) (width 0.25) (layer "B.Cu") (net 15))
   (segment (start 24.4 -52.9504) (end 24.6745 -52.6759) (width 0.25) (layer "B.Cu") (net 15))
   (segment (start 38.1105 -51.9105) (end 38.725 -52.525) (width 0.25) (layer "B.Cu") (net 15))
-  (segment (start 18.794294 -29.275) (end 21.413357 -31.894063) (width 0.25) (layer "B.Cu") (net 15))
-  (segment (start 13.5 -30.25) (end 14.475 -29.275) (width 0.25) (layer "B.Cu") (net 15))
+  (segment (start 13.5 -30.25) (end 14.725 -29.025) (width 0.25) (layer "B.Cu") (net 15))
+  (segment (start 18.825 -29.025) (end 21.413357 -31.613357) (width 0.25) (layer "B.Cu") (net 15))
   (segment (start 35.134501 -51.9105) (end 38.1105 -51.9105) (width 0.25) (layer "B.Cu") (net 15))
   (segment (start 25.525 -54) (end 26.275 -54.75) (width 0.25) (layer "F.Cu") (net 17))
@@
   (segment (start 68.725 -16.95) (end 68.725 -14.625) (width 0.25) (layer "B.Cu") (net 40))
   (segment (start 68.725 -14.625) (end 67.7 -13.6) (width 0.25) (layer "B.Cu") (net 40))
+  (zone (net 10) (net_name "GND") (layers "F&B.Cu") (hatch edge 0.5)
+    (connect_pads (clearance 0.508))
+    (min_thickness 0.25) (filled_areas_thickness no)
+    (fill yes (thermal_gap 0.5) (thermal_bridge_width 0.5))
+    (polygon
+      (pts
+        (xy -21 -76.6)
+        (xy 102.5 -79.8)
+        (xy 93.9 23.5)
+        (xy -33.2 17.4)
+        (xy -21.4 -76.8)
+      )
+    )
+  )
 )
