File: production/pcbs/5.0/right/right.kicad_pcb (KiCad board)
At the start: 2 copper layers, 90 x 71 mm, 43 parts, among them T1 Flactyl 5.0 (right)

Commit message: Versions
Parts:
- T1: moved to F.Cu
Connections:
- ROT1 pad 1: C0_R3D -> C0
- ROT1 pad 2: C0 -> C0_R3D
Routing:
- net C4_R1: track 156.1 -> 0.00 mm, vias 3 -> 0
- net C4_R0: track 150.7 -> 0.00 mm, vias 7 -> 0
- net R2: track 0.00 -> 141.4 mm, vias 0 -> 8
- net P1: track 141.4 -> 0.00 mm, vias 8 -> 0
- net R0: track 9.80 -> 150.7 mm, vias 0 -> 7
- net C4_R1D: track 127.0 -> 9.80 mm, vias 9 -> 0
- net R1: track 11.6 -> 127.0 mm, vias 0 -> 9
- net R3: track 29.5 -> 124.0 mm, vias 2 -> 4
- net RAW: track 0.00 -> 93.5 mm, vias 0 -> 2
- net GND: track 93.5 -> 0.00 mm, vias 2 -> 0
- net VCC: track 91.5 -> 0.00 mm, vias 2 -> 0
- net C0: track 71.7 -> 156.1 mm, vias 2 -> 3
- net P2: track 0.00 -> 71.7 mm, vias 0 -> 2
- net C0_R3D: track 80.2 -> 11.6 mm, vias 3 -> 0
- net C6: track 0.00 -> 60.3 mm, vias 0 -> 2
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Other:
- net class Default removed

Commit message: Add right pcb
Routing:
- net C0: track 156.1 -> 157.7 mm
- net P2: track 71.7 -> 72.5 mm
- net RST: track 86.9 -> 87.6 mm
