File: production/pcbs/5.0/thumb3/thumb3.kicad_pcb (KiCad board)
At the start: 2 copper layers, 20 x 51 mm, 12 parts, among them T1 Flactyl 5.0 (thumb3), T2 x, T3 y

Commit message: iceberg-ploopy
Routing:
- net C5: track 45.0 -> 62.0 mm
Changed lines of the file:
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@@
 (gr_arc (start -8.5 -41) (end -8.5 -42.5) (angle -90) (layer Eco1.User) (width 0.15))
 (gr_arc (start -8.5 7) (end -10 7) (angle -90) (layer Eco1.User) (width 0.15))
-(gr_line (start -9 -6) (end 2 -6) (angle 90) (layer Eco1.User) (width 0.15))
-(gr_line (start 2 -6) (end 2 -28) (angle 90) (layer Eco1.User) (width 0.15))
-(gr_line (start 2 -28) (end -9 -28) (angle 90) (layer Eco1.User) (width 0.15))
-(gr_line (start -9 -28) (end -9 -6) (angle 90) (layer Eco1.User) (width 0.15))
+(gr_line (start -8.5 -16.5) (end 1.5 -16.5) (angle 90) (layer Eco1.User) (width 0.15))
+(gr_line (start 1.5 -16.5) (end 1.5 -26.5) (angle 90) (layer Eco1.User) (width 0.15))
+(gr_line (start 1.5 -26.5) (end -8.5 -26.5) (angle 90) (layer Eco1.User) (width 0.15))
+(gr_line (start -8.5 -26.5) (end -8.5 -16.5) (angle 90) (layer Eco1.User) (width 0.15))
+(gr_circle (center -5 -8.5) (end -3.9 -8.5) (layer Eco1.User) (width 0.15))
 (gr_circle (center 5 -25.5) (end 6.1 -25.5) (layer Eco1.User) (width 0.15))
 (gr_line (start -9 8.5) (end 9 8.5) (angle 90) (layer Eco2.User) (width 0.15))
@@
   (segment (start -7.446751 -23.5) (end -7 -23.5) (width 0.25) (layer "B.Cu") (net 1))
   (segment (start -8.275 -22.671751) (end -7.446751 -23.5) (width 0.25) (layer "B.Cu") (net 1))
+  (segment (start -8.275 3.75) (end -8.275 -13.25) (width 0.25) (layer "B.Cu") (net 1))
   (segment (start 4.2 -41.825) (end -4.65 -41.825) (width 0.25) (layer "B.Cu") (net 1))
   (segment (start 8.275 -37.75) (end 4.2 -41.825) (width 0.25) (layer "B.Cu") (net 1))
