File: production/pcbs/misc/cirque-connector/cirque-connector.kicad_pcb (KiCad board)
At the start: 2 copper layers, 15 x 34 mm, 6 parts, among them J1 Conn_01x12_Socket, J2 Conn_01x12_Socket

Commit message: Some more connectors.
Other:
- board text added: "3V GND SDA SCL B1 B2 B3 SI DR SS SO SCK"
Changed lines of the file:
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@@
     (property "ki_keywords" "connector")
     (attr smd)
-    (fp_text reference "J1" (at -0.232 -2.448 90) (layer "F.SilkS")
+    (fp_text reference "J1" (at -0.2 2.362 90) (layer "F.SilkS")
         (effects (font (size 1.143 1.143) (thickness 0.152)) (justify right))
     )
@@
   (gr_line (start 28 51) (end 28 85)
     (stroke (width 0.05) (type default)) (layer "Edge.Cuts"))
+  (gr_text "3V\n\nGND\n\nSDA\n\nSCL\n\nB1\n\nB2\n\nB3\n\nSI\n\nDR\n\nSS\n\nSO\n\nSCK" (at 39 83.8) (layer "B.SilkS" knockout)
+    (effects (font (size 0.8 0.8) (thickness 0.2) bold) (justify left bottom mirror))
+  )
+  (gr_text "3V\n\nGND\n\nSDA\n\nSCL\n\nB1\n\nB2\n\nB3\n\nSI\n\nDR\n\nSS\n\nSO\n\nSCK" (at 37.2 83.6) (layer "F.SilkS")
+    (effects (font (size 0.8 0.8) (thickness 0.2) bold) (justify left bottom))
+  )
   (segment (start 35.724 61.95) (end 35.724 60.256) (width 0.2) (layer "F.Cu") (net 1))
   (segment (start 35.724 60.256) (end 41 54.98) (width 0.2) (layer "F.Cu") (net 1))
